File: mechanical_keyboard_mk1/key_matrix.sch (KiCad schematic (older format))
At the start: 28 parts

Commit message: Update
Parts:
- added D14, D15, D16, D17, D18, D19, D20, D21, D22, D23, D24, D25, D26, D27, D28, D29, D30, D31, D32, D33, D34, D35, D36, D37, D38, D39, D40, D41, D42, D43, D44, D45, D46, D47, D48, D49, D50, D51, D52, D53, D54, D55, D56, D57, D58, D59, D60: 1N4148, mechanical_keyboard_mk1:D_DO-35_SOD27_P7.62mm_Horizontal, symbol Diode:1N4148
- added R_COL_0, R_COL_1, R_COL_10, R_COL_11, R_COL_12, R_COL_13, R_COL_2, R_COL_3, R_COL_4, R_COL_5, R_COL_6, R_COL_7, R_COL_8, R_COL_9: 10k, Resistors_THT:R_Axial_DIN0207_L6.3mm_D2.5mm_P7.62mm_Horizontal, symbol Device:R_US
- added SW_"_1U1, SW_,_1U1, SW_._1U1, SW_/_1U1, SW_;_1U1, SW_A_1U1, SW_B_1U1, SW_CTRL_1U1, SW_C_1U1, SW_D_1U1, SW_E_1U1, SW_F_1U1, SW_G_1U1, SW_H_1U1, SW_I_1U1, SW_J_1U1, SW_K_1U1, SW_L_1U1, SW_M_1U1, SW_N_1U1, SW_O_1U1, SW_PRTSC_1U1, SW_P_1U1, SW_Q_1U1, SW_R_1U1, SW_S_1U1, SW_T_1U1, SW_U_1U1, SW_V_1U1, SW_WINR_1U1, SW_W_1U1, SW_X_1U1, SW_Y_1U1, SW_Z_1U1, SW_[_1U1, SW_]_1U1: SW_SPST, Button_Switch_Keyboard:SW_Cherry_MX_1.00u_PCB, symbol Switch:SW_SPST
- added SW_ALTR_1.25U1, SW_OS_1.25U1: SW_SPST, Button_Switch_Keyboard:SW_Cherry_MX_1.25u_PCB, symbol Switch:SW_SPST
- added SW_CAPS_1.75: SW_SPST, Button_Switch_Keyboard:SW_Cherry_MX_1.75u_PCB, symbol Switch:SW_SPST
- added SW_ENTER_2.25U1, SW_SHIFT_2.25U1: SW_SPST, Button_Switch_Keyboard:SW_Cherry_MX_2.25u_PCB, symbol Switch:SW_SPST
- added SW_FN_1.5U1, SW_MENU_1.5U1, SW_TAB_1.5U1, SW_\_1.5U1: SW_SPST, Button_Switch_Keyboard:SW_Cherry_MX_1.50u_PCB, symbol Switch:SW_SPST
- added SW_SHIFT_2.75U1: SW_SPST, Button_Switch_Keyboard:SW_Cherry_MX_2.75u_PCB, symbol Switch:SW_SPST
- added SW_SPC_6.5U1: SW_SPST, mechanical_keyboard_mk1:SW_Cherry_MX_6.5u_PCB, symbol Switch:SW_SPST
- D0, D1, D10, D11, D12, D13, D2, D3, D4, D5, D6, D7, D8, D9: footprint Diode_THT:D_DO-35_SOD27_P7.62mm_Horizontal -> mechanical_keyboard_mk1:D_DO-35_SOD27_P7.62mm_Horizontal
Connections:
- net COL_0: now also D14.1 (K), D28.1 (K), D41.1 (K), D53.1 (K), R_COL_0.1
- net COL_1: now also D15.1 (K), D29.1 (K), D42.1 (K), D54.1 (K), R_COL_1.1
- net COL_10: now also D24.1 (K), D38.1 (K), D51.1 (K), D58.1 (K), R_COL_10.1
- net COL_11: now also D25.1 (K), D39.1 (K), D52.1 (K), D59.1 (K), R_COL_11.1
- net COL_12: now also D26.1 (K), D40.1 (K), D60.1 (K), R_COL_12.1
- net COL_13: now also D27.1 (K), R_COL_13.1
- net COL_2: now also D16.1 (K), D30.1 (K), D43.1 (K), D55.1 (K), R_COL_2.1
- net COL_3: now also D17.1 (K), D31.1 (K), D44.1 (K), D56.1 (K), R_COL_3.1
- net COL_4: now also D18.1 (K), D32.1 (K), D45.1 (K), R_COL_4.1
- net COL_5: now also D19.1 (K), D33.1 (K), D46.1 (K), R_COL_5.1
- net COL_6: now also D20.1 (K), D34.1 (K), D47.1 (K), R_COL_6.1
- net COL_7: now also D21.1 (K), D35.1 (K), D48.1 (K), R_COL_7.1
- net COL_8: now also D22.1 (K), D36.1 (K), D49.1 (K), R_COL_8.1
- net COL_9: now also D23.1 (K), D37.1 (K), D50.1 (K), D57.1 (K), R_COL_9.1
- new net: D14.2 (A), SW_TAB_1.5U1.2 (B)
- new net: D15.2 (A), SW_Q_1U1.2 (B)
- new net: D16.2 (A), SW_W_1U1.2 (B)
- new net: D17.2 (A), SW_E_1U1.2 (B)
- new net: D18.2 (A), SW_R_1U1.2 (B)
- new net: D19.2 (A), SW_T_1U1.2 (B)
- new net: D20.2 (A), SW_Y_1U1.2 (B)
- new net: D21.2 (A), SW_U_1U1.2 (B)
- new net: D22.2 (A), SW_I_1U1.2 (B)
- new net: D23.2 (A), SW_O_1U1.2 (B)
- new net: D24.2 (A), SW_P_1U1.2 (B)
- new net: D25.2 (A), SW_[_1U1.2 (B)
- new net: D26.2 (A), SW_]_1U1.2 (B)
- new net: D27.2 (A), SW_\_1.5U1.2 (B)
- new net: D28.2 (A), SW_CAPS_1.75.2 (B)
- new net: D29.2 (A), SW_A_1U1.2 (B)
- new net: D30.2 (A), SW_S_1U1.2 (B)
- new net: D31.2 (A), SW_D_1U1.2 (B)
- new net: D32.2 (A), SW_F_1U1.2 (B)
- new net: D33.2 (A), SW_G_1U1.2 (B)
- new net: D34.2 (A), SW_H_1U1.2 (B)
- new net: D35.2 (A), SW_J_1U1.2 (B)
- new net: D36.2 (A), SW_K_1U1.2 (B)
- new net: D37.2 (A), SW_L_1U1.2 (B)
- new net: D38.2 (A), SW_;_1U1.2 (B)
- new net: D39.2 (A), SW_"_1U1.2 (B)
- new net: D40.2 (A), SW_ENTER_2.25U1.2 (B)
- new net: D41.2 (A), SW_SHIFT_2.25U1.2 (B)
- new net: D42.2 (A), SW_Z_1U1.2 (B)
- new net: D43.2 (A), SW_X_1U1.2 (B)
- new net: D44.2 (A), SW_C_1U1.2 (B)
- new net: D45.2 (A), SW_V_1U1.2 (B)
- new net: D46.2 (A), SW_B_1U1.2 (B)
- new net: D47.2 (A), SW_N_1U1.2 (B)
- new net: D48.2 (A), SW_M_1U1.2 (B)
- new net: D49.2 (A), SW_,_1U1.2 (B)
- new net: D50.2 (A), SW_._1U1.2 (B)
- new net: D51.2 (A), SW_/_1U1.2 (B)
- new net: D52.2 (A), SW_SHIFT_2.75U1.2 (B)
- new net: D53.2 (A), SW_FN_1.5U1.2 (B)
- new net: D54.2 (A), SW_CTRL_1U1.2 (B)
- new net: D55.2 (A), SW_OS_1.25U1.2 (B)
- new net: D56.2 (A), SW_SPC_6.5U1.2 (B)
- new net: D57.2 (A), SW_ALTR_1.25U1.2 (B)
- new net: D58.2 (A), SW_PRTSC_1U1.2 (B)
- new net: D59.2 (A), SW_WINR_1U1.2 (B)
- new net: D60.2 (A), SW_MENU_1.5U1.2 (B)
- new net GND: R_COL_0.2, R_COL_1.2, R_COL_10.2, R_COL_11.2, R_COL_12.2, R_COL_13.2, R_COL_2.2, R_COL_3.2, R_COL_4.2, R_COL_5.2, R_COL_6.2, R_COL_7.2, R_COL_8.2, R_COL_9.2
- new net ROW_1: SW_E_1U1.1 (A), SW_I_1U1.1 (A), SW_O_1U1.1 (A), SW_P_1U1.1 (A), SW_Q_1U1.1 (A), SW_R_1U1.1 (A), SW_TAB_1.5U1.1 (A), SW_T_1U1.1 (A), SW_U_1U1.1 (A), SW_W_1U1.1 (A), SW_Y_1U1.1 (A), SW_[_1U1.1 (A), SW_\_1.5U1.1 (A), SW_]_1U1.1 (A)
- new net ROW_2: SW_"_1U1.1 (A), SW_;_1U1.1 (A), SW_A_1U1.1 (A), SW_CAPS_1.75.1 (A), SW_D_1U1.1 (A), SW_ENTER_2.25U1.1 (A), SW_F_1U1.1 (A), SW_G_1U1.1 (A), SW_H_1U1.1 (A), SW_J_1U1.1 (A), SW_K_1U1.1 (A), SW_L_1U1.1 (A), SW_S_1U1.1 (A)
- new net ROW_3: SW_,_1U1.1 (A), SW_._1U1.1 (A), SW_/_1U1.1 (A), SW_B_1U1.1 (A), SW_C_1U1.1 (A), SW_M_1U1.1 (A), SW_N_1U1.1 (A), SW_SHIFT_2.25U1.1 (A), SW_SHIFT_2.75U1.1 (A), SW_V_1U1.1 (A), SW_X_1U1.1 (A), SW_Z_1U1.1 (A)
- new net ROW_4: SW_ALTR_1.25U1.1 (A), SW_CTRL_1U1.1 (A), SW_FN_1.5U1.1 (A), SW_MENU_1.5U1.1 (A), SW_OS_1.25U1.1 (A), SW_PRTSC_1U1.1 (A), SW_SPC_6.5U1.1 (A), SW_WINR_1U1.1 (A)
Other:
- moved on the sheet: D10, D11, D8, D9, SW_-_1U1, SW_0_1U1, SW_8_1U1, SW_9_1U1
