File: mechanical_keyboard_mk1/mechanical_keyboard_mk1.kicad_pcb (KiCad board)
At the start: 2 copper layers, 28 parts

Commit message: Update
Parts:
- removed D0, D1, D10, D11, D12, D13, D2, D3, D4, D5, D6, D7, D8, D9: 1N4148, Diode_THT:D_DO-35_SOD27_P7.62mm_Horizontal
- removed SW_-_1U1, SW_0_1U1, SW_1_1U1, SW_2_1U1, SW_3_1U1, SW_5_1U1, SW_6_1U1, SW_7_1U1, SW_8_1U1, SW_9_1U1, SW_=_1U1, SW_TIL_1U1: SW_SPST, Button_Switch_Keyboard:SW_Cherry_MX_1.00u_PCB
- removed SW_BKSP_2U1: SW_SPST, Button_Switch_Keyboard:SW_Cherry_MX_2.00u_PCB
- added D41: 1N4148, mechanical_keyboard_mk1:D_DO-35_SOD27_P7.62mm_Horizontal, F.Cu at (21.5, 93.3)
- added D42: 1N4148, mechanical_keyboard_mk1:D_DO-35_SOD27_P7.62mm_Horizontal, F.Cu at (64.4, 93.3)
- added D43: 1N4148, mechanical_keyboard_mk1:D_DO-35_SOD27_P7.62mm_Horizontal, F.Cu at (83.4, 93.3)
- added D44: 1N4148, mechanical_keyboard_mk1:D_DO-35_SOD27_P7.62mm_Horizontal, F.Cu at (102.5, 93.3)
- added D45: 1N4148, mechanical_keyboard_mk1:D_DO-35_SOD27_P7.62mm_Horizontal, F.Cu at (121.5, 93.3)
- added D46: 1N4148, mechanical_keyboard_mk1:D_DO-35_SOD27_P7.62mm_Horizontal, F.Cu at (140.6, 93.3)
- added D47: 1N4148, mechanical_keyboard_mk1:D_DO-35_SOD27_P7.62mm_Horizontal, F.Cu at (159.6, 93.3)
- added D48: 1N4148, mechanical_keyboard_mk1:D_DO-35_SOD27_P7.62mm_Horizontal, F.Cu at (178.7, 93.3)
- added D49: 1N4148, mechanical_keyboard_mk1:D_DO-35_SOD27_P7.62mm_Horizontal, F.Cu at (197.7, 93.3)
- added D50: 1N4148, mechanical_keyboard_mk1:D_DO-35_SOD27_P7.62mm_Horizontal, F.Cu at (216.8, 93.3)
- added D51: 1N4148, mechanical_keyboard_mk1:D_DO-35_SOD27_P7.62mm_Horizontal, F.Cu at (235.8, 93.3)
- added D52: 1N4148, mechanical_keyboard_mk1:D_DO-35_SOD27_P7.62mm_Horizontal, F.Cu at (254.9, 93.3)
- added D53: 1N4148, mechanical_keyboard_mk1:D_DO-35_SOD27_P7.62mm_Horizontal, F.Cu at (21.6, 112.4)
- added D54: 1N4148, mechanical_keyboard_mk1:D_DO-35_SOD27_P7.62mm_Horizontal, F.Cu at (50.2, 112.4)
- added D55: 1N4148, mechanical_keyboard_mk1:D_DO-35_SOD27_P7.62mm_Horizontal, F.Cu at (69.2, 112.4)
- added D56: 1N4148, mechanical_keyboard_mk1:D_DO-35_SOD27_P7.62mm_Horizontal, F.Cu at (93.1, 112.4)
- added D57: 1N4148, mechanical_keyboard_mk1:D_DO-35_SOD27_P7.62mm_Horizontal, F.Cu at (216.9, 112.4)
- added D58: 1N4148, mechanical_keyboard_mk1:D_DO-35_SOD27_P7.62mm_Horizontal, F.Cu at (240.7, 112.4)
- added D59: 1N4148, mechanical_keyboard_mk1:D_DO-35_SOD27_P7.62mm_Horizontal, F.Cu at (259.7, 112.4)
- added D60: 1N4148, mechanical_keyboard_mk1:D_DO-35_SOD27_P7.62mm_Horizontal, F.Cu at (278.7, 112.4)
- added R_COL_0: 10k, Resistors_THT:R_Axial_DIN0207_L6.3mm_D2.5mm_P7.62mm_Horizontal, B.Cu at (21.6, 120.3)
- added R_COL_1: 10k, Resistors_THT:R_Axial_DIN0207_L6.3mm_D2.5mm_P7.62mm_Horizontal, B.Cu at (50.2, 120.3)
- added R_COL_10: 10k, Resistors_THT:R_Axial_DIN0207_L6.3mm_D2.5mm_P7.62mm_Horizontal, B.Cu at (235.7, 120.3)
- added R_COL_11: 10k, Resistors_THT:R_Axial_DIN0207_L6.3mm_D2.5mm_P7.62mm_Horizontal, B.Cu at (254.9, 120.3)
- added R_COL_12: 10k, Resistors_THT:R_Axial_DIN0207_L6.3mm_D2.5mm_P7.62mm_Horizontal, B.Cu at (270.6, 120.3)
- added R_COL_13: 10k, Resistors_THT:R_Axial_DIN0207_L6.3mm_D2.5mm_P7.62mm_Horizontal, B.Cu at (285.1, 120.3)
- added R_COL_2: 10k, Resistors_THT:R_Axial_DIN0207_L6.3mm_D2.5mm_P7.62mm_Horizontal, B.Cu at (69.2, 120.3)
- added R_COL_3: 10k, Resistors_THT:R_Axial_DIN0207_L6.3mm_D2.5mm_P7.62mm_Horizontal, B.Cu at (93.0, 120.3)
- added R_COL_4: 10k, Resistors_THT:R_Axial_DIN0207_L6.3mm_D2.5mm_P7.62mm_Horizontal, B.Cu at (121.5, 120.2)
- added R_COL_5: 10k, Resistors_THT:R_Axial_DIN0207_L6.3mm_D2.5mm_P7.62mm_Horizontal, B.Cu at (140.5, 120.2)
- added R_COL_6: 10k, Resistors_THT:R_Axial_DIN0207_L6.3mm_D2.5mm_P7.62mm_Horizontal, B.Cu at (169.5, 120.3)
- added R_COL_7: 10k, Resistors_THT:R_Axial_DIN0207_L6.3mm_D2.5mm_P7.62mm_Horizontal, B.Cu at (182.4, 120.3)
- added R_COL_8: 10k, Resistors_THT:R_Axial_DIN0207_L6.3mm_D2.5mm_P7.62mm_Horizontal, B.Cu at (197.7, 120.3)
- added R_COL_9: 10k, Resistors_THT:R_Axial_DIN0207_L6.3mm_D2.5mm_P7.62mm_Horizontal, B.Cu at (216.8, 120.3)
- added SW_: , Button_Switch_Keyboard:SW_Cherry_MX_1.00u_PCB, F.Cu at (257.6, 64.1)
- added SW_,_1U1: SW_SPST, Button_Switch_Keyboard:SW_Cherry_MX_1.00u_PCB, F.Cu at (209.8, 83.2)
- added SW_._1U1: SW_SPST, Button_Switch_Keyboard:SW_Cherry_MX_1.00u_PCB, F.Cu at (228.9, 83.2)
- added SW_/_1U1: SW_SPST, Button_Switch_Keyboard:SW_Cherry_MX_1.00u_PCB, F.Cu at (247.9, 83.2)
- added SW_;_1U1: SW_SPST, Button_Switch_Keyboard:SW_Cherry_MX_1.00u_PCB, F.Cu at (238.5, 64.1)
- added SW_ALTR_1.25U1: SW_SPST, Button_Switch_Keyboard:SW_Cherry_MX_1.25u_PCB, F.Cu at (231.3, 102.2)
- added SW_A_1U1: SW_SPST, Button_Switch_Keyboard:SW_Cherry_MX_1.00u_PCB, F.Cu at (66.9, 64.1)
- added SW_B_1U1: SW_SPST, Button_Switch_Keyboard:SW_Cherry_MX_1.00u_PCB, F.Cu at (152.7, 83.2)
- added SW_CAPS_1.75: SW_SPST, Button_Switch_Keyboard:SW_Cherry_MX_1.75u_PCB, F.Cu at (40.8, 64.1)
- added SW_CTRL_1U1: SW_SPST, Button_Switch_Keyboard:SW_Cherry_MX_1.00u_PCB, F.Cu at (62.2, 102.2)
- added SW_C_1U1: SW_SPST, Button_Switch_Keyboard:SW_Cherry_MX_1.00u_PCB, F.Cu at (114.6, 83.2)
- added SW_D_1U1: SW_SPST, Button_Switch_Keyboard:SW_Cherry_MX_1.00u_PCB, F.Cu at (105.2, 64.1)
- added SW_ENTER_2.25U1: SW_SPST, Button_Switch_Keyboard:SW_Cherry_MX_2.25u_PCB, F.Cu at (288.5, 64.1)
- added SW_FN_1.5U1: SW_SPST, Button_Switch_Keyboard:SW_Cherry_MX_1.50u_PCB, F.Cu at (38.4, 102.2)
- added SW_F_1U1: SW_SPST, Button_Switch_Keyboard:SW_Cherry_MX_1.00u_PCB, F.Cu at (124.2, 64.1)
- added SW_G_1U1: SW_SPST, Button_Switch_Keyboard:SW_Cherry_MX_1.00u_PCB, F.Cu at (143.3, 64.1)
- added SW_H_1U1: SW_SPST, Button_Switch_Keyboard:SW_Cherry_MX_1.00u_PCB, F.Cu at (162.3, 64.1)
- added SW_J_1U1: SW_SPST, Button_Switch_Keyboard:SW_Cherry_MX_1.00u_PCB, F.Cu at (181.4, 64.1)
- added SW_K_1U1: SW_SPST, Button_Switch_Keyboard:SW_Cherry_MX_1.00u_PCB, F.Cu at (200.4, 64.1)
- added SW_L_1U1: SW_SPST, Button_Switch_Keyboard:SW_Cherry_MX_1.00u_PCB, F.Cu at (219.5, 64.1)
- added SW_MENU_1.5U1: SW_SPST, Button_Switch_Keyboard:SW_Cherry_MX_1.50u_PCB, F.Cu at (295.5, 102.2)
- added SW_M_1U1: SW_SPST, Button_Switch_Keyboard:SW_Cherry_MX_1.00u_PCB, F.Cu at (190.8, 83.2)
- added SW_N_1U1: SW_SPST, Button_Switch_Keyboard:SW_Cherry_MX_1.00u_PCB, F.Cu at (171.7, 83.2)
- added SW_OS_1.25U1: SW_SPST, Button_Switch_Keyboard:SW_Cherry_MX_1.25u_PCB, F.Cu at (83.7, 102.2)
- added SW_PRTSC_1U1: SW_SPST, Button_Switch_Keyboard:SW_Cherry_MX_1.00u_PCB, F.Cu at (252.7, 102.2)
- added SW_SHIFT_2.25U1: SW_SPST, Button_Switch_Keyboard:SW_Cherry_MX_2.25u_PCB, F.Cu at (45.5, 83.2)
- added SW_SHIFT_2.75U1: SW_SPST, Button_Switch_Keyboard:SW_Cherry_MX_2.75u_PCB, F.Cu at (283.6, 83.2)
- added SW_SPC_6.5U1: SW_SPST, mechanical_keyboard_mk1:SW_Cherry_MX_6.5u_PCB, F.Cu at (157.5, 102.2)
- added SW_S_1U1: SW_SPST, Button_Switch_Keyboard:SW_Cherry_MX_1.00u_PCB, F.Cu at (86.1, 64.1)
- added SW_V_1U1: SW_SPST, Button_Switch_Keyboard:SW_Cherry_MX_1.00u_PCB, F.Cu at (133.6, 83.2)
- added SW_WINR_1U1: SW_SPST, Button_Switch_Keyboard:SW_Cherry_MX_1.00u_PCB, F.Cu at (271.7, 102.2)
- added SW_X_1U1: SW_SPST, Button_Switch_Keyboard:SW_Cherry_MX_1.00u_PCB, F.Cu at (95.5, 83.2)
- added SW_Z_1U1: SW_SPST, Button_Switch_Keyboard:SW_Cherry_MX_1.00u_PCB, F.Cu at (76.5, 83.2)
- moved SW_4_1U1 16.2 mm to (109.9, 26.0)
Routing:
- net /key_matrix/ROW_4: track 0.00 -> 259.3 mm
- net /key_matrix/ROW_1: track 0.00 -> 257.2 mm
- net /key_matrix/ROW_2: track 0.00 -> 247.8 mm
- net /key_matrix/ROW_3: track 0.00 -> 238.1 mm
- net /key_matrix/ROW_0: track 0.00 -> 228.6 mm
- net /key_matrix/COL_0: track 0.00 -> 82.6 mm
- net Net-(D14-Pad2): track 0.00 -> 10.5 mm
- net Net-(D54-Pad2): track 0.00 -> 5.72 mm
- net Net-(D3-Pad2): track 0.00 -> 5.72 mm
- net Net-(D2-Pad2): track 0.00 -> 5.72 mm
- net Net-(D16-Pad2): track 0.00 -> 5.72 mm
- net Net-(D15-Pad2): track 0.00 -> 5.72 mm
- net Net-(D0-Pad2): track 0.00 -> 5.71 mm
- net Net-(D1-Pad2): track 0.00 -> 5.71 mm
Other:
- board outline added: 304.8 x 114.3 mm
- net class Default: clearance 0.2 -> 0.254; trace_width 0.25 -> 0.4064; via_dia 0.8 -> 0.6096; via_drill 0.4 -> 0.4064
- rule trace_clearance: 0.2 -> 0.254
