File: mechanical_keyboard_mk1/mechanical_keyboard_mk1.sch (KiCad schematic (older format))
At the start: 0 parts

Commit message: Update
Changed lines of the file:
@@
 EESchema Schematic File Version 4
+LIBS:mechanical_keyboard_mk1-cache
 EELAYER 29 0
 EELAYER END
@@
 $EndDescr
 $Sheet
-S 6500 1200 1050 1100
+S 6500 1000 550  2150
 U 5CF479B5
 F0 "key_matrix" 50
 F1 "key_matrix.sch" 50
+F2 "ROW_0" I L 6500 1050 50
+F3 "COL_0" I L 6500 1750 50
+F4 "COL_1" I L 6500 1850 50
+F5 "COL_2" I L 6500 1950 50
+F6 "COL_3" I L 6500 2050 50
+F7 "COL_4" I L 6500 2150 50
+F8 "COL_5" I L 6500 2250 50
+F9 "COL_6" I L 6500 2350 50
+F10 "COL_7" I L 6500 2450 50
+F11 "COL_8" I L 6500 2550 50
+F12 "COL_9" I L 6500 2650 50
+F13 "COL_10" I L 6500 2750 50
+F14 "COL_11" I L 6500 2850 50
+F15 "COL_12" I L 6500 2950 50
+F16 "COL_13" I L 6500 3050 50
+F17 "ROW_1" I L 6500 1150 50
+F18 "ROW_2" I L 6500 1250 50
+F19 "ROW_3" I L 6500 1350 50
+F20 "ROW_4" I L 6500 1450 50
 $EndSheet
 $EndSCHEMATC
